File: KiCad/Radargun.kicad_pcb (KiCad board)
At the start: 2 copper layers, 70 x 45 mm, 56 parts, among them J1 UART_PROG, J2 TM1637, J3 TP4056 module, J4 HB100 Radar, Q1 AO3401A, Q2 2N7002, SW1 RESET, SW2 BOOT, SW3 SW_Push, SW4 POWER_SW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

Commit message: PCB placement update
Parts:
- moved C4 172.2 mm to (150.2, 66.2)
- moved C3 171.7 mm to (150.2, 64.0)
- moved C5 171.0 mm to (150.2, 71.0)
- moved R7 163.5 mm to (174.2, 80.8), turned to 180 degrees
- moved R6 152.7 mm to (150.2, 68.8), turned to 180 degrees
- moved J1 138.3 mm to (174.2, 65.9)
- moved SW3 122.3 mm to (139.5, 78.2)
- moved L1 117.2 mm to (114.8, 94.5), turned to 180 degrees
- moved U3 107.6 mm to (114.8, 101.0)
- moved SW1 99.4 mm to (110.5, 65.5)
- moved SW2 98.2 mm to (110.5, 75.5)
- moved R2 92.4 mm to (111.5, 103.2), turned to 90 degrees
- moved R1 92.1 mm to (114.8, 103.8), turned to 180 degrees
- moved H1 86.5 mm to (128.2, 161.8)
- moved U1 44.0 mm to (162.2, 72.3)
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Other:
- outline, holes or cut-outs redrawn
